File: hardware/flash.kicad_sch (KiCad schematic)
At the start: 6 parts, among them U3 W25Q128JVSIQ

Commit message: Add MFR numbers to the passive components
Parts:
- C27: JLCPCB Part # (none) -> C15849
- C28: JLCPCB Part # (none) -> C14663
- R17: JLCPCB Part # (none) -> C98220
- R18: JLCPCB Part # (none) -> C22548
Changed lines of the file:
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@@
+			)
+		)
+		(property "JLCPCB Part #" "C98220"
+			(at 119.38 92.71 0)
+			(effects
+				(font
+					(size 1.27 1.27)
+				)
+				(hide yes)
 			)
 		)
@@
 			)
 		)
+		(property "JLCPCB Part #" "C15849"
+			(at 175.26 104.14 0)
+			(effects
+				(font
+					(size 1.27 1.27)
+				)
+				(hide yes)
+			)
+		)
 		(pin "1"
 		)
@@
 			)
 		)
+		(property "JLCPCB Part #" "C22548"
+			(at 119.38 102.87 0)
+			(effects
+				(font
+					(size 1.27 1.27)
+				)
+				(hide yes)
+			)
+		)
 		(pin "1"
 		)
@@
 			)
 		)
+		(property "JLCPCB Part #" "C14663"
+			(at 185.42 104.14 0)
+			(effects
+				(font
+					(size 1.27 1.27)
+				)
+				(hide yes)
+			)
+		)
