File: hardware/usb.kicad_sch (KiCad schematic)
At the start: 17 parts, among them J7 TYPE-C-31-M-13C, U5 USBLC6-2SC6, U6 NCP1117LPST33T3G

Commit message: Add MFR numbers to the passive components
Parts:
- C31, C33: JLCPCB Part # (none) -> C14663
- C32, C34: JLCPCB Part # (none) -> C19702
- R20, R21: JLCPCB Part # (none) -> C2907044
- R22: JLCPCB Part # (none) -> C114627
- R23: JLCPCB Part # (none) -> C98220
Changed lines of the file:
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@@
+			)
+		)
+		(property "JLCPCB Part #" "C98220"
+			(at 158.75 104.14 0)
+			(effects
+				(font
+					(size 1.27 1.27)
+				)
+				(hide yes)
 			)
 		)
@@
 			)
 		)
+		(property "JLCPCB Part #" "C14663"
+			(at 147.32 96.52 0)
+			(effects
+				(font
+					(size 1.27 1.27)
+				)
+				(hide yes)
+			)
+		)
 		(pin "1"
 		)
@@
 			)
 		)
+		(property "JLCPCB Part #" "C114627"
+			(at 158.75 96.52 0)
+			(effects
+				(font
+					(size 1.27 1.27)
+				)
+				(hide yes)
+			)
+		)
 		(pin "1"
 		)
@@
 					(size 1.27 1.27)
 				)
+			)
+		)
+		(property "JLCPCB Part #" "C14663"
+			(at 218.44 96.52 0)
+			(effects
+				(font
+					(size 1.27 1.27)
+				)
+				(hide yes)
 			)
 		)
@@
 			)
 		)
+		(property "JLCPCB Part #" "C19702"
+			(at 231.14 96.52 0)
+			(effects
+				(font
+					(size 1.27 1.27)
+				)
+				(hide yes)
+			)
+		)
 		(pin "1"
 		)
@@
 			)
 		)
+		(property "JLCPCB Part #" "C2907044"
+			(at 99.06 99.06 90)
+			(effects
+				(font
+					(size 1.27 1.27)
+				)
+				(hide yes)
+			)
+		)
 		(pin "1"
 		)
@@
 					(size 1.27 1.27)
 				)
+			)
+		)
+		(property "JLCPCB Part #" "C19702"
+			(at 189.23 96.52 0)
+			(effects
+				(font
+					(size 1.27 1.27)
+				)
+				(hide yes)
 			)
 		)
@@
 			)
 		)
+		(property "JLCPCB Part #" "C2907044"
+			(at 99.06 96.52 90)
+			(effects
+				(font
+					(size 1.27 1.27)
+				)
+				(hide yes)
+			)
+		)

Commit message: Add test points to LED DIN and DOUT
Parts:
- renumbered TP8 to TP10, TP9 to TP11, TP7 to TP9
Changed lines of the file:
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@@
 		(on_board yes)
 		(dnp no)
-		(property "Reference" "TP9"
+		(property "Reference" "TP11"
 			(at 233.68 90.17 0)
 			(effects
@@
 			(project "katia"
 				(path "/4cc5d416-57f5-4147-8183-e03ae6b1198a/089db7cd-2934-428b-a62a-55e0735649ba/92c7d305-84cf-4400-bd59-4f28ecb1b049"
-					(reference "TP9")
-					(unit 1)
-				)
-				(path "/4cc5d416-57f5-4147-8183-e03ae6b1198a/50d96a5e-3d25-4129-9495-15388c76587f/109c87e7-e271-4132-84ce-4a528ef290f8"
-					(reference "TP12")
+					(reference "TP11")
+					(unit 1)
+				)
+				(path "/4cc5d416-57f5-4147-8183-e03ae6b1198a/50d96a5e-3d25-4129-9495-15388c76587f/109c87e7-e271-4132-84ce-4a528ef290f8"
+					(reference "TP16")
 					(unit 1)
 				)
@@
 		(on_board yes)
 		(dnp no)
-		(property "Reference" "TP8"
+		(property "Reference" "TP10"
 			(at 191.77 90.17 0)
 			(effects
@@
 			(project "katia"
 				(path "/4cc5d416-57f5-4147-8183-e03ae6b1198a/089db7cd-2934-428b-a62a-55e0735649ba/92c7d305-84cf-4400-bd59-4f28ecb1b049"
-					(reference "TP8")
-					(unit 1)
-				)
-				(path "/4cc5d416-57f5-4147-8183-e03ae6b1198a/50d96a5e-3d25-4129-9495-15388c76587f/109c87e7-e271-4132-84ce-4a528ef290f8"
-					(reference "TP11")
+					(reference "TP10")
+					(unit 1)
+				)
+				(path "/4cc5d416-57f5-4147-8183-e03ae6b1198a/50d96a5e-3d25-4129-9495-15388c76587f/109c87e7-e271-4132-84ce-4a528ef290f8"
+					(reference "TP15")
 					(unit 1)
 				)
@@
 		(on_board yes)
 		(dnp no)
-		(property "Reference" "TP7"
+		(property "Reference" "TP9"
 			(at 73.66 129.54 0)
 			(effects
@@
 			(project "katia"
 				(path "/4cc5d416-57f5-4147-8183-e03ae6b1198a/089db7cd-2934-428b-a62a-55e0735649ba/92c7d305-84cf-4400-bd59-4f28ecb1b049"
-					(reference "TP7")
-					(unit 1)
-				)
-				(path "/4cc5d416-57f5-4147-8183-e03ae6b1198a/50d96a5e-3d25-4129-9495-15388c76587f/109c87e7-e271-4132-84ce-4a528ef290f8"
-					(reference "TP10")
-					(unit 1)
-				)
+					(reference "TP9")
+					(unit 1)
+				)
+				(path "/4cc5d416-57f5-4147-8183-e03ae6b1198a/50d96a5e-3d25-4129-9495-15388c76587f/109c87e7-e271-4132-84ce-4a528ef290f8"
+					(reference "TP14")
+					(unit 1)
+				)

Commit message: Replace Schottky diode with higher-current variant
Parts:
- D3: value VS-10BQ015HM3/5BT -> CDBM240L-HF; JLCPCB Part # C23848 -> C3012684
Changed lines of the file:
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@@
 			)
 		)
-		(property "Value" "VS-10BQ015HM3/5BT"
+		(property "Value" "CDBM240L-HF"
 			(at 170.18 87.63 0)
 			(effects
@@
 			)
 		)
-		(property "Datasheet" "https://lcsc.com/datasheet/lcsc_datasheet_2410010303_onsemi-MBR0520LT1G_C23848.pdf"
+		(property "Datasheet" "https://www.lcsc.com/datasheet/C3012684.pdf"
 			(at 170.18 91.44 90)
 			(effects
@@
 			)
 		)
-		(property "JLCPCB Part #" "C23848"
+		(property "JLCPCB Part #" "C3012684"
 			(at 170.18 91.44 0)
 			(effects
